File: Hardware/dummyload.brd (EAGLE design)
At the start: 73.7 x 53.7 mm, 47 parts, among them IC1 MCP1700, Q1 IRFB7430PBF, SW1 SWITCH-B3U-1110-BOSS, U1 ATMEGA32U4-AU, U2 LMP2022, U3 MCP3426, U4 MAX5812, X1 USB-MINI/MICRO-4S-4LEGS, Y1 16MHz

Commit message: updated to use 0.5 ohm cur sense resistor
Parts:
- R-SENSE: value 1R -> 0R5
Changed lines of the file:
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@@
 <layer number="21" name="tPlace" color="7" fill="1" visible="yes" active="yes"/>
 <layer number="22" name="bPlace" color="7" fill="1" visible="no" active="yes"/>
-<layer number="23" name="tOrigins" color="15" fill="1" visible="no" active="yes"/>
+<layer number="23" name="tOrigins" color="15" fill="1" visible="yes" active="yes"/>
 <layer number="24" name="bOrigins" color="15" fill="1" visible="no" active="yes"/>
 <layer number="25" name="tNames" color="7" fill="1" visible="yes" active="yes"/>
@@
 <attribute name="NAME" x="46.779" y="31.654" size="0.8128" layer="25" ratio="10" rot="R270"/>
 </element>
-<element name="R-SENSE" library="minilab" package="D2PACK" value="1R" x="66.4" y="26.86" smashed="yes" rot="R270">
+<element name="R-SENSE" library="minilab" package="D2PACK" value="0R5" x="66.4" y="26.86" smashed="yes" rot="R270">
 <attribute name="NAME" x="62.698" y="33.443" size="0.8128" layer="25" ratio="10"/>
 </element>
